File: Hardware/AlarmMain/AlarmMain.kicad_pcb (KiCad board)
At the start: 2 copper layers, 218 parts, among them J1 debugWIRE, J10 I2C, J11 ICSP, J12 AUX, J13 RS485, J14 PWR, J15 BATT, J16 12V, J17 DI1, J18 DI2, J19 DI3, J2 OP1, J20 DI4, J21 DI5, J22 DI6, J23 DI7, J24 DI8, J3 OP3, J4 DI9, J5 DI10, J6 OP2, J7 OP4, J8 DI11, J9 DI12, Q1 STP40NF03L, Q2 STP40NF03L, Q3 STP40NF03L, Q4 STP40NF03L, Q5 IRF9540N, Q6 IRF540N, Q7 BC337, SW1 RESET, U1 ATmega328P-PU, U10 LM317_TO-220, U11 LM324, U12 7805, U13 LM339, U14 LM339, U15 LM339, U16 LM339, U2 LM339, U3 LM339, U4 MCP23017_SP, U5 DS18B20, U6 MCP7940N-xSN, U7 STTS75, U8 STWD100, U9 MAX483E, Y1 20Mhz, Y2 32.768k

Commit message: PCB progressive updates
Parts:
- added C16: 100n, Capacitor_THT:C_Disc_D4.3mm_W1.9mm_P5.00mm, F.Cu at (49.4, 2.26)
- moved R85 122.9 mm to (137.5, 129.5), turned to 270 degrees
- moved C14 115.7 mm to (180.3, 65.8)
- moved R93 111.7 mm to (133.3, 53.6)
- moved R83 110.4 mm to (125.2, 129.5), turned to 270 degrees
- moved R57 106.2 mm to (64.1, 129.5), turned to 270 degrees
- moved C15 105.1 mm to (161.2, 65.8)
- moved R69 98.5 mm to (128.1, 77.4)
- moved R81 97.6 mm to (113.0, 129.5), turned to 270 degrees
- moved R99 90.9 mm to (114.2, 61.2), turned to 270 degrees
- moved C55 86.4 mm to (142.2, 65.8)
- moved R59 84.1 mm to (76.4, 129.5), turned to 270 degrees
- moved R7 68.2 mm to (149.7, 129.5), turned to 270 degrees
- moved C54 57.4 mm to (123.1, 65.8)
- moved C52 57.0 mm to (104.1, 65.8)
- moved R25 54.8 mm to (174.1, 129.5), turned to 270 degrees
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Routing:
- net GND: track 1010.9 -> 1122.6 mm
- net VBAT_SUP: track 318.9 -> 423.2 mm
- net +5V: track 350.1 -> 420.6 mm
- net DI4: track 63.0 -> 68.5 mm
- net DI6: track 64.1 -> 69.2 mm
- net Net-(C16-Pad1): track 14.7 -> 19.6 mm
- net VBAT_ADJ: track 42.8 -> 47.2 mm
- net DI8: track 72.2 -> 76.6 mm
- net DI2: track 69.2 -> 73.3 mm
- net DI3: track 49.6 -> 53.6 mm
- net DI5: track 52.5 -> 56.1 mm
- net DI1: track 58.6 -> 62.2 mm
- net DI7: track 60.9 -> 57.5 mm

Commit message: Furst python layout scripts
Parts:
- moved R78 131.3 mm to (184.5, 72.7), turned to 270 degrees
- moved R11 129.6 mm to (84.5, 57.5), turned to 270 degrees
- moved R70 126.4 mm to (184.5, 65.1), turned to 90 degrees
- moved R21 124.9 mm to (84.5, 72.7), turned to 270 degrees
- moved R102 114.2 mm to (199.1, 75.2), turned to 270 degrees
- moved R94 108.9 mm to (199.1, 70.2), turned to 270 degrees
- moved R26 108.4 mm to (99.1, 65.1)
- moved R92 106.1 mm to (159.1, 70.2), turned to 270 degrees
- moved R8 103.1 mm to (84.5, 67.6), turned to 270 degrees
- moved R29 102.9 mm to (99.1, 57.5), turned to 270 degrees
- moved R32 97.6 mm to (119.1, 70.2), turned to 270 degrees
- moved C14 93.2 mm to (88.0, 78.7)
- moved R15 92.4 mm to (84.5, 62.5), turned to 270 degrees
- moved U2 92.1 mm to (88.0, 60.0)
- moved R62 90.1 mm to (184.5, 70.2), turned to 90 degrees
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Routing:
- net GND: track 1122.6 -> 0.00 mm, vias 16 -> 0
- net VBAT_SUP: track 423.2 -> 0.00 mm
- net +5V: track 420.6 -> 0.00 mm, vias 3 -> 0
- net VBAT_TEST: track 160.8 -> 0.00 mm
- net VBAT_DIS: track 146.5 -> 0.00 mm
- net VIN: track 132.1 -> 0.00 mm
- net RESET: track 112.7 -> 0.00 mm
- net VPWR_MON: track 95.9 -> 0.00 mm
- net SDA: track 93.6 -> 0.00 mm
- net DO1: track 81.1 -> 0.00 mm
- net SCL: track 81.0 -> 0.00 mm
- net DI8: track 76.6 -> 0.00 mm
- net DI2: track 73.3 -> 0.00 mm
- net DI6: track 69.2 -> 0.00 mm
- net VBAT_MON: track 68.8 -> 0.00 mm
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
Commit message: Progressive layout
Parts:
- moved C39 59.6 mm to (86.7, 16.6)
- moved C11 55.4 mm to (139.8, 20.6)
- moved C36 50.5 mm to (76.8, 27.0), turned to 90 degrees
- moved C38 42.1 mm to (94.8, 36.6)
- moved C37 41.8 mm to (103.9, 36.4)
- moved C42 41.0 mm to (115.1, 36.1)
- moved C35 41.0 mm to (124.5, 36.1)
- moved R10 18.5 mm to (98.5, 52.6), turned to 270 degrees
- moved R16 18.5 mm to (98.5, 47.5), turned to 270 degrees
- moved R56 18.5 mm to (118.5, 52.6), turned to 270 degrees
- moved R58 18.5 mm to (138.5, 52.6), turned to 270 degrees
- moved R60 18.5 mm to (158.5, 52.6), turned to 270 degrees
- moved R62 18.5 mm to (178.5, 52.6), turned to 270 degrees
- moved R67 18.5 mm to (118.5, 47.5), turned to 270 degrees
- moved R68 18.5 mm to (138.5, 47.5), turned to 270 degrees
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Connections:
- R11 pad 2: DI9 -> DI1
- R12 pad 2: DI10 -> DI3
- R29 pad 2: DI11 -> DI2
- R30 pad 2: DI12 -> DI4
- R63 pad 2: DI1 -> DI5
- R64 pad 2: DI2 -> DI6
- R65 pad 2: DI3 -> DI7
- R66 pad 2: DI4 -> DI8
- R87 pad 2: DI5 -> DI9
- R88 pad 2: DI6 -> DI10
- R89 pad 2: DI7 -> DI11
- R90 pad 2: DI8 -> DI12
- U13 pad 1: DI1 -> DI5
- U13 pad 13: DI5 -> DI9
- U13 pad 14: DI5 -> DI9
- U13 pad 2: DI1 -> DI5
- U14 pad 1: DI2 -> DI6
- U14 pad 13: DI6 -> DI10
- U14 pad 14: DI6 -> DI10
- U14 pad 2: DI2 -> DI6
- U15 pad 1: DI3 -> DI7
- U15 pad 13: DI7 -> DI11
- U15 pad 14: DI7 -> DI11
- U15 pad 2: DI3 -> DI7
- U16 pad 1: DI4 -> DI8
- U16 pad 13: DI8 -> DI12
- U16 pad 14: DI8 -> DI12
- U16 pad 2: DI4 -> DI8
- U2 pad 1: DI9 -> DI1
- U2 pad 13: DI11 -> DI2
- U2 pad 14: DI11 -> DI2
- U2 pad 2: DI9 -> DI1
- U3 pad 1: DI10 -> DI3
- U3 pad 13: DI12 -> DI4
- U3 pad 14: DI12 -> DI4
- U3 pad 2: DI10 -> DI3

Commit message: Input connector order change
Parts:
- moved C12 110.0 mm to (67.3, 71.5)
- moved J8 110.0 mm to (62.2, 85.0)
- moved R25 110.0 mm to (63.3, 74.5)
- moved R33 110.0 mm to (67.3, 74.5)
- moved C13 97.8 mm to (91.7, 71.5)
- moved J4 97.8 mm to (50.0, 85.0)
- moved R27 97.8 mm to (87.7, 74.5)
- moved R34 97.8 mm to (91.7, 74.5)
- moved C8 97.8 mm to (55.1, 71.5)
- moved J9 97.8 mm to (86.7, 85.0)
- moved R17 97.8 mm to (55.1, 74.5)
- moved R7 97.8 mm to (51.1, 74.5)
- moved C47 85.5 mm to (177.3, 71.5)
- moved C9 85.5 mm to (79.5, 71.5)
- moved R18 85.5 mm to (79.5, 74.5)
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Connections:
- R11 pad 2: DI1 -> DI9
- R12 pad 2: DI3 -> DI10
- R29 pad 2: DI2 -> DI11
- R30 pad 2: DI4 -> DI12
- R63 pad 2: DI5 -> DI1
- R64 pad 2: DI6 -> DI2
- R65 pad 2: DI7 -> DI3
- R66 pad 2: DI8 -> DI4
- R87 pad 2: DI9 -> DI5
- R88 pad 2: DI10 -> DI6
- R89 pad 2: DI11 -> DI7
- R90 pad 2: DI12 -> DI8
- U13 pad 1: DI5 -> DI1
- U13 pad 13: DI9 -> DI5
- U13 pad 14: DI9 -> DI5
- U13 pad 2: DI5 -> DI1
- U14 pad 1: DI6 -> DI2
- U14 pad 13: DI10 -> DI6
- U14 pad 14: DI10 -> DI6
- U14 pad 2: DI6 -> DI2
- U15 pad 1: DI7 -> DI3
- U15 pad 13: DI11 -> DI7
- U15 pad 14: DI11 -> DI7
- U15 pad 2: DI7 -> DI3
- U16 pad 1: DI8 -> DI4
- U16 pad 13: DI12 -> DI8
- U16 pad 14: DI12 -> DI8
- U16 pad 2: DI8 -> DI4
- U2 pad 1: DI1 -> DI9
- U2 pad 13: DI2 -> DI11
- U2 pad 14: DI2 -> DI11
- U2 pad 2: DI1 -> DI9
- U3 pad 1: DI3 -> DI10
- U3 pad 13: DI4 -> DI12
- U3 pad 14: DI4 -> DI12
- U3 pad 2: DI3 -> DI10

Commit message: Completed tracks first pass
Parts:
- moved C37 15.8 mm to (99.9, 21.1), turned to 270 degrees
- moved R35 0.92 mm to (139.2, 33.8)
Connections:
- U4 pad 22: DI12 -> DI1
- U4 pad 23: DI9 -> DI2
- U4 pad 24: DI11 -> DI6
- U4 pad 6: DI1 -> DI12
- U4 pad 7: DI6 -> DI11
- U4 pad 8: DI2 -> DI9
Routing:
- net GND: track 0.00 -> 1666.0 mm, vias 0 -> 1
- net VBAT_SUP: track 0.00 -> 833.6 mm, vias 0 -> 2
- net +5V: track 0.00 -> 437.0 mm
- net VBAT_DIS: track 0.00 -> 297.1 mm
- net VIN: track 0.00 -> 194.0 mm, vias 0 -> 1
- net VBAT_TEST: track 0.00 -> 143.0 mm, vias 0 -> 1
- net RESET: track 0.00 -> 117.3 mm
- net VBAT: track 0.00 -> 109.3 mm
- net SCL: track 0.00 -> 97.7 mm
- net VPWR_MON: track 0.00 -> 97.5 mm, vias 0 -> 5
- net SDA: track 0.00 -> 86.1 mm
- net DO1: track 0.00 -> 78.8 mm
- net DI9: track 0.00 -> 75.5 mm
- net DI11: track 0.00 -> 69.7 mm
- net VBAT_MON: track 0.00 -> 69.0 mm
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
Commit message: Rework to 4 layers
Parts:
- removed D2: LED, LED_THT:LED_D5.0mm
- removed R38: 4K7, Resistor_THT:R_Axial_DIN0204_L3.6mm_D1.6mm_P2.54mm_Vertical
- removed R4: 330R, Resistor_THT:R_Axial_DIN0204_L3.6mm_D1.6mm_P2.54mm_Vertical
- added C17: 100n, Capacitor_THT:C_Disc_D4.3mm_W1.9mm_P5.00mm, F.Cu at (211.4, 19.6)
- added C56: 100n, Capacitor_THT:C_Disc_D4.3mm_W1.9mm_P5.00mm, F.Cu at (211.4, 16.3)
- added J25: RS485 2, TerminalBlock_Phoenix:TerminalBlock_Phoenix_MKDS-1,5-4-5.08_1x04_P5.08mm_Horizontal, F.Cu at (220.0, 34.1)
- J13: value RS485 -> RS485 1
- U5: value DS18B20 -> MAX483E; footprint Package_TO_SOT_THT:TO-92_Inline -> Package_SO:SOIC-8_3.9x4.9mm_P1.27mm
- moved U5 68.7 mm to (209.0, 26.0)
- moved C42 49.7 mm to (77.8, 3.35)
- moved C35 36.2 mm to (93.5, 17.3)
- moved C23 13.7 mm to (211.4, -4.78), turned to 180 degrees
- moved R14 13.4 mm to (201.0, 59.0), turned to 180 degrees
- moved R13 13.4 mm to (201.0, 46.8), turned to 180 degrees
- moved R24 13.4 mm to (201.0, 83.4), turned to 180 degrees
- moved R23 13.3 mm to (201.0, 71.2), turned to 180 degrees
- moved R20 13.2 mm to (200.9, 78.3)
- moved R6 13.2 mm to (200.9, 53.9)
- moved R5 13.2 mm to (201.0, 41.7)
- moved J2 13.2 mm to (220.0, 46.7)
- moved J3 13.2 mm to (220.0, 59.0)
- moved J6 13.2 mm to (220.0, 71.2)
- moved J7 13.2 mm to (220.0, 83.4)
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Connections:
- C32 pad 1: Net-(C32-Pad1) -> +12V
- C33 pad 1: Net-(C32-Pad1) -> +12V
- D5 pad 1: Net-(C32-Pad1) -> +12V
- J12 pad 3: +5V -> TEMP_INT
- J13 pad 1: VBAT_SUP -> +12V
- J16 pad 2: Net-(C32-Pad1) -> +12V
- J2 pad 1: VBAT_SUP -> +12V
- J3 pad 1: VBAT_SUP -> +12V
- J6 pad 1: VBAT_SUP -> +12V
- J7 pad 1: VBAT_SUP -> +12V
- U1 pad 15: LED2 -> RTS_2
- U1 pad 23: VBAT_DIS -> VBAT_TEST
- U1 pad 24: VBAT_TEST -> VBAT_DIS
- U1 pad 25: VBAT_MON -> VPWR_MON
- U1 pad 26: VPWR_MON -> VBAT_MON
- U1 pad 5: TEMP_INT -> RXD_2
- U1 pad 6: ONEWIRE -> TXD_2
- U4 pad 1: DI8 -> DO4
- U4 pad 2: DI4 -> DO3
- U4 pad 25: DO1 -> DI3
- U4 pad 26: DO2 -> DI7
- U4 pad 27: DO3 -> DI4
- U4 pad 28: DO4 -> DI8
- U4 pad 3: DI7 -> DO2
- U4 pad 4: DI3 -> DO1
- U5 pad 1: GND -> RXD_2
- U5 pad 2: ONEWIRE -> RTS_2
- U5 pad 3: +5V -> RTS_2
Routing:
- net +12V: track 0.00 -> 421.0 mm
- net VBAT_DIS: track 297.1 -> 178.1 mm
- net RTS_2: track 0.00 -> 99.3 mm
- net TXD_2: track 0.00 -> 73.8 mm
- net VBAT_SUP: track 833.6 -> 760.9 mm, vias 2 -> 0
- net RXD_2: track 0.00 -> 67.5 mm
- net +5V: track 437.0 -> 495.3 mm, vias 0 -> 1
- net VIN: track 194.0 -> 149.3 mm, vias 1 -> 0
- net VBAT: track 109.3 -> 142.7 mm
- net Net-(C32-Pad1): track 31.9 -> 0.00 mm
- net VBAT_MON: track 69.0 -> 97.7 mm
- net VBAT_TEST: track 143.0 -> 168.1 mm, vias 1 -> 0
- net VPWR_MON: track 97.5 -> 119.4 mm, vias 5 -> 0
- net ONEWIRE: track 17.3 -> 0.00 mm
- net DI3: track 39.8 -> 23.3 mm
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- added copper zone on POWER_SIG_3RD, net +5V
- added copper zone on GND_SIG_2ND, net GND
- added copper zone on B.Cu, net VBAT_SUP
- removed copper zone on B.Cu, net GND
Other:
- board outline added: 209.2 x 93.2 mm
- copper layers 2 -> 4
- board text added: "+12V"
- board text added: "+12V A B COM"
- board text added: "BATT"
- board text added: "COM +VE"
- board text added: "COM INP"
- board text added: "COM OUT"
- board text added: "INP 1"
- board text added: "INP 10"
- board text added: "INP 11"
- board text added: "INP 12"
- board text added: "INP 2"
- board text added: "INP 3"
- board text added: "INP 4"
- board text added: "INP 5"
- board text added: "INP 6"
- board text added: "INP 7"
- board text added: "INP 8"
- board text added: "INP 9"
- board text added: "INP INP"
- board text added: "IO-MODULE-12I4O"
- board text added: "MEKATROL"
- board text added: "OUT 1"
- board text added: "PWR IN"
- board text added: "RS485 DEVICE"
- board text added: "RS485 EXTERNAL"
- board text added: "V1.0 (22 May 2021)"

Commit message: Moved files
Parts:
- added R2: 4K7, Resistor_THT:R_Axial_DIN0204_L3.6mm_D1.6mm_P2.54mm_Vertical, F.Cu at (22.5, 58.5)
- R43: footprint Resistor_THT:R_Axial_DIN0204_L3.6mm_D1.6mm_P2.54mm_Vertical -> Resistor_THT:R_Box_L8.4mm_W2.5mm_P5.08mm
- R44: value 10K -> 100K
- R45: value 10K -> 200R
- moved R42 6.46 mm to (18.4, 62.2), turned to 90 degrees
- moved R44 5.58 mm to (23.8, 62.9)
- moved R43 3.03 mm to (19.1, 55.3)
- moved R45 2.21 mm to (26.4, 59.1)
- moved Q7 0.97 mm to (23.8, 52.2)
Connections:
- R42 pad 1: Net-(Q7-Pad1) -> Net-(Q5-Pad1)
- R42 pad 2: VBAT -> VBAT_SUP
- R44 pad 1: Net-(Q5-Pad1) -> GND
- R44 pad 2: Net-(Q7-Pad1) -> Net-(Q7-Pad2)
Routing:
- net Net-(Q7-Pad2): track 3.89 -> 12.4 mm
- net VBAT_SUP: track 760.9 -> 768.7 mm
- net Net-(Q5-Pad1): track 5.68 -> 11.7 mm
- net Net-(Q7-Pad1): track 8.78 -> 4.28 mm
- net VBAT_DIS: track 178.1 -> 176.0 mm
- net VBAT: track 142.7 -> 141.3 mm
- net Net-(Q6-Pad2): track 3.82 -> 4.49 mm
Other:
- board size 209.2 x 93.2 mm -> 244 x 109 mm

Commit message: Fixes to PCB silkscreen
Other:
- board text added: "+5V"
- board text added: "GND"
- board text added: "MFP"
- board text added: "MISO"
- board text added: "MOSI"
- board text added: "OUT 2"
- board text added: "OUT 3"
- board text added: "OUT 4"
- board text added: "RST"
- board text added: "SCK"
- board text added: "SCL"
- board text added: "SDA"
- board text added: "TMP INT"
- board text added: "V1.1 (30 June 2021)"
- board text removed: "V1.0 (22 May 2021)"
